File: hardware/electrical/sensor.kicad_sch (KiCad schematic)
At the start: 10 parts

Commit message: Update schematic to include regulators and switches, update render
Parts:
- renumbered C1 to C21, C2 to C22, C3 to C23, C4 to C24, C5 to C25, C6 to C26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
Connections:
- net +1.8V: no longer C21.1, C22.1, R3.2, R5.2, U5.5 (VDDIO)
- new net VDDIO: C21.1, C22.1, R3.2, R5.2, U5.5 (VDDIO)
